Commit message: Removed 8th dof for now and made sure urdf works in gazebo. Also copied some files over from homework for trajectory code

File: urdf/tennis.urdf (robot description, URDF)
Before this commit: robot SevenDOF, 30 links, 29 joints
Links:
- removed link base
- removed link handbase
- removed link link0
- removed link racket_collision
- added link racketv, mass 0.16; visual cylinder length=0.01 radius=.25
- link racket: mass 0.16 -> None; geometry collision cylinder length=0.01 radius=.2
Joints:
- removed joint attach-base
- removed joint attach-handbase
- removed joint attach-racket_collision
- removed joint theta0
- added joint attach-racketv: type fixed, parent tip, child racketv
- joint attach-motor1: parent link0 -> world
- joint attach-mount1: parent link0 -> world
- joint final: origin xyz=0 0.25 0 rpy=1.5708 0 3.1416 -> xyz=0 0.25 0 rpy=0 0 0
- joint theta1: parent link0 -> world
