Commit message: urdf working in gazebo

File: 8DOF_arm/urdf/8DOF_arm.urdf (robot description, URDF)
Before this commit: robot 8DOF_arm, 9 links, 8 joints
Links:
- added link motor1, mass 2.0; visual cylinder length=0.02 radius=0.005
- added link motor2, mass 2.0; visual cylinder length=0.02 radius=0.005
- added link motor3, mass 2.0; visual cylinder length=0.02 radius=0.005
- added link motor4, mass 2.0; visual cylinder length=0.02 radius=0.005
- added link motor5, mass 2.0; visual cylinder length=0.02 radius=0.005
- added link motor6, mass 2.0; visual cylinder length=0.02 radius=0.005
- added link motor7, mass 2.0; visual cylinder length=0.02 radius=0.005
- added link motor8, mass 2.0; visual cylinder length=0.1 radius=0.005
- added link mount1, mass 0.2; visual cylinder length=0.02 radius=0.002
- added link mount2, mass 0.2; visual cylinder length=0.02 radius=0.002
- added link mount3, mass 0.2; visual cylinder length=0.02 radius=0.002
- added link mount4, mass 0.2; visual cylinder length=0.02 radius=0.002
- added link mount5, mass 0.2; visual cylinder length=0.02 radius=0.002
- added link mount6, mass 0.2; visual cylinder length=0.02 radius=0.002
- added link mount7, mass 0.2; visual cylinder length=0.02 radius=0.002
- added link mount8, mass 0.2; visual cylinder length=0.1 radius=0.002
- added link tip
- added link world
Joints:
- removed joint base_pin
- removed joint first_link
- removed joint first_pin
- removed joint second_link
- removed joint second_pin
- removed joint tennis_pin
- removed joint tennis_racket
- removed joint third_link
- added joint attach-motor1: type fixed, parent base_link, child motor1
- added joint attach-motor2: type fixed, parent base_pin, child motor2
- added joint attach-motor3: type fixed, parent first_link, child motor3
- added joint attach-motor4: type fixed, parent first_pin, child motor4
- added joint attach-motor5: type fixed, parent second_link, child motor5
- added joint attach-motor6: type fixed, parent second_pin, child motor6
- added joint attach-motor7: type fixed, parent third_link, child motor7
- added joint attach-motor8: type fixed, parent tennis_pin, child motor8
- added joint attach-mount1: type fixed, parent base_link, child mount1
- added joint attach-mount2: type fixed, parent base_pin, child mount2
- added joint attach-mount3: type fixed, parent first_link, child mount3
- added joint attach-mount4: type fixed, parent first_pin, child mount4
- added joint attach-mount5: type fixed, parent second_link, child mount5
- added joint attach-mount6: type fixed, parent second_pin, child mount6
- added joint attach-mount7: type fixed, parent third_link, child mount7
- added joint attach-mount8: type fixed, parent tennis_pin, child mount8
- added joint final: type fixed, parent tennis_racket, child tip, origin xyz=0 0.02 0 rpy=0 0 0
- added joint theta1: type continuous, parent base_link, child base_pin, origin xyz=0 0 0.0698499999999998 rpy=1.5707963267949 0 0, axis 0 1 0
- added joint theta2: type continuous, parent base_pin, child first_link, origin xyz=0 0.0635 0 rpy=1.5707963267949 1.5707963267949 0, axis 1 0 0
- added joint theta3: type continuous, parent first_link, child first_pin, origin xyz=0 -0.094412 0 rpy=0 0 -1.5708, axis 1 0 0
- added joint theta4: type continuous, parent first_pin, child second_link, origin xyz=0.0380999999999999 0 0 rpy=1.5707963267949 0 -1.5707963267949, axis 1 0 0
- added joint theta5: type continuous, parent second_link, child second_pin, origin xyz=0 -0.094412 0 rpy=1.5708 0 -1.5708, axis 1 0 0
- added joint theta6: type continuous, parent second_pin, child third_link, origin xyz=0.0381 0 0 rpy=1.5707963267949 0 -1.5707963267949, axis 1 0 0
- added joint theta7: type continuous, parent third_link, child tennis_pin, origin xyz=0 0.094412 0 rpy=0 1.5708 0, axis 0 1 0
- added joint theta8: type continuous, parent tennis_pin, child tennis_racket, origin xyz=0 0.0571499999999999 0 rpy=0 -0.661454620295037 1.5707963267949, axis 0 1 0
- added joint worldfixed: type fixed, parent world, child base_link, origin xyz=0 0 0 rpy=0 0 0

Commit message: fixing rviz launch and collisions for urdf

File: 8DOF_arm/urdf/8DOF_arm.urdf (robot description, URDF)
Before this commit: robot 8DOF_arm, 27 links, 26 joints
Links:
- link base_link: geometry visual mesh filename=package://8DOF_arm/meshes/base_link.STL
- link base_pin: geometry visual mesh filename=package://8DOF_arm/meshes/base_pin.STL
- link first_link: geometry visual mesh filename=package://8DOF_arm/meshes/first_link.STL
- link first_pin: geometry visual mesh filename=package://8DOF_arm/meshes/first_pin.STL
- link second_link: geometry visual mesh filename=package://8DOF_arm/meshes/second_link.STL
- link second_pin: geometry visual mesh filename=package://8DOF_arm/meshes/second_pin.STL
- link tennis_pin: geometry visual mesh filename=package://8DOF_arm/meshes/tennis_pin.STL
- link tennis_racket: geometry visual mesh filename=package://8DOF_arm/meshes/tennis_racket.STL
- link third_link: geometry visual mesh filename=package://8DOF_arm/meshes/third_link.STL
